File: hw/DRV8825.sch (KiCad schematic (older format))
At the start: 15 parts, among them P5 CONN_2, P6 CONN_2, U4 MCP47X6, U5 DRV8825

Commit message: Added additional caps to the DAC on the stepper feedback
Parts:
- added C19, C22: 10uF, symbol CP1
- added C20, C21, C23: 100nF, symbol C
- added R13: 1M, symbol R
- C10: value 0.1uF -> 100nF
- R5: value 500k -> 1M
Connections:
- wire segments 62 -> 68
Changed lines of the file:
@@
 P 5750 2900
 F 0 "C10" H 5750 3000 40  0000 L CNN
-F 1 "0.1uF" H 5756 2815 40  0000 L CNN
+F 1 "100nF" H 5756 2815 40  0000 L CNN
 F 2 "" H 5788 2750 30  0000 C CNN
 F 3 "" H 5750 2900 60  0000 C CNN
@@
 $EndComp
 Wire Wire Line
-	3100 3850 3550 3850
-Text Label 3250 3200 1    60   ~ 0
+	3100 3850 3800 3850
+Text Label 3350 3200 1    60   ~ 0
 3V3Ref
 $Comp
@@
 Connection ~ 1800 4150
 Wire Wire Line
-	2000 3750 1800 3750
+	1250 3750 2000 3750
 Wire Wire Line
 	1800 3750 1800 3700
@@
 P 3250 3500
 F 0 "R5" V 3330 3500 40  0000 C CNN
-F 1 "500k" V 3257 3501 40  0000 C CNN
+F 1 "1M" V 3257 3501 40  0000 C CNN
 F 2 "" V 3180 3500 30  0000 C CNN
 F 3 "" H 3250 3500 30  0000 C CNN
@@
 $EndComp
 Wire Wire Line
-	3100 3750 3250 3750
-Wire Wire Line
-	3250 3250 3250 2900
+	3100 3750 4550 3750
+Wire Wire Line
+	3350 3250 3350 2900
 $Comp
 L CONN_2 P5
@@
 Text Label 4550 1450 0    60   ~ 0
 VMOT
+$Comp
+L C C20
+U 1 1 539F6E90
+P 1550 3950
+F 0 "C20" H 1550 4050 40  0000 L CNN
+F 1 "100nF" H 1556 3865 40  0000 L CNN
+F 2 "" H 1588 3800 30  0000 C CNN
+F 3 "" H 1550 3950 60  0000 C CNN
+	1    1550 3950
+	1    0    0    -1
+$EndComp
+$Comp
+L CP1 C19
+U 1 1 539F6EA4
+P 1250 3950
+F 0 "C19" H 1300 4050 50  0000 L CNN
+F 1 "10uF" H 1300 3850 50  0000 L CNN
+F 2 "" H 1250 3950 60  0000 C CNN
+F 3 "" H 1250 3950 60  0000 C CNN
+	1    1250 3950
+	1    0    0    -1
+$EndComp
+Connection ~ 1800 3750
+Connection ~ 1550 3750
+Wire Wire Line
+	1250 4150 1550 4150
+Wire Wire Line
+	1400 4150 1400 4250
+Connection ~ 1400 4150
+$Comp
+L GND #PWR035
+U 1 1 539F6FF5
+P 1400 4250
+F 0 "#PWR035" H 1400 4250 30  0001 C CNN
+F 1 "GND" H 1400 4180 30  0001 C CNN
+F 2 "" H 1400 4250 60  0000 C CNN
+F 3 "" H 1400 4250 60  0000 C CNN
+	1    1400 4250
+	1    0    0    -1
+$EndComp
+$Comp
+L C C23
+U 1 1 539F7008
+P 4550 3950
+F 0 "C23" H 4550 4050 40  0000 L CNN
+F 1 "100nF" H 4556 3865 40  0000 L CNN
+F 2 "" H 4588 3800 30  0000 C CNN
+F 3 "" H 4550 3950 60  0000 C CNN
+	1    4550 3950
+	1    0    0    -1
+$EndComp
+$Comp
+L CP1 C22
+U 1 1 539F700E
+P 4250 3950
+F 0 "C22" H 4300 4050 50  0000 L CNN
+F 1 "10uF" H 4300 3850 50  0000 L CNN
+F 2 "" H 4250 3950 60  0000 C CNN
+F 3 "" H 4250 3950 60  0000 C CNN
+	1    4250 3950
+	1    0    0    -1
+$EndComp
+Connection ~ 4550 3750
+Wire Wire Line
+	4250 4150 4550 4150
+Wire Wire Line
+	4400 4150 4400 4250
+Connection ~ 4400 4150
+$Comp
+L GND #PWR036
+U 1 1 539F7018
+P 4400 4250
+F 0 "#PWR036" H 4400 4250 30  0001 C CNN
+F 1 "GND" H 4400 4180 30  0001 C CNN
+F 2 "" H 4400 4250 60  0000 C CNN
+F 3 "" H 4400 4250 60  0000 C CNN
+	1    4400 4250
+	1    0    0    -1
+$EndComp
+Connection ~ 3250 3750
+Connection ~ 4250 3750
+$Comp
+L C C21
+U 1 1 539F70C5
+P 3800 4050
+F 0 "C21" H 3800 4150 40  0000 L CNN
+F 1 "100nF" H 3806 3965 40  0000 L CNN
+F 2 "" H 3838 3900 30  0000 C CNN
+F 3 "" H 3800 4050 60  0000 C CNN
+	1    3800 4050
+	1    0    0    -1
+$EndComp
+Wire Wire Line
+	3800 4250 3800 4300
+$Comp
+L GND #PWR037
+U 1 1 539F717A
+P 3800 4300
+F 0 "#PWR037" H 3800 4300 30  0001 C CNN
+F 1 "GND" H 3800 4230 30  0001 C CNN
+F 2 "" H 3800 4300 60  0000 C CNN
+F 3 "" H 3800 4300 60  0000 C CNN
+	1    3800 4300
+	1    0    0    -1
+$EndComp
+$Comp
+L R R13
+U 1 1 539F7448
+P 3450 3500
+F 0 "R13" V 3530 3500 40  0000 C CNN
+F 1 "1M" V 3457 3501 40  0000 C CNN
+F 2 "" V 3380 3500 30  0000 C CNN
+F 3 "" H 3450 3500 30  0000 C CNN
+	1    3450 3500
+	1    0    0    -1
+$EndComp
+Wire Wire Line
+	3250 3250 3450 3250
+Connection ~ 3350 3250
+Connection ~ 3450 3750
 $EndSCHEMATC
