File: hw/nema17_driver.sch (KiCad schematic (older format))
At the start: 14 parts, among them P1 CONN_6, P2 CONN_4, P3 CONN_6, P4 CONN_2, SW1 SW_PUSH, U1 ATMEGA328P, X1 16Mhz

Commit message: Added additional caps to the DAC on the stepper feedback
Parts:
- C1, C4: value 0.1uF -> 100nF
Changed lines of the file:
@@
 F0 "Power" 50
 F1 "Power.sch" 50
-F4 "45V" I L 10050 1850 60
+F2 "45V" I L 10050 1850 60
 $EndSheet
 Text Label 9700 750  0    60   ~ 0
@@
 P 3250 3650
 F 0 "C1" H 3250 3750 40  0000 L CNN
-F 1 "0.1uF" H 3256 3565 40  0000 L CNN
+F 1 "100nF" H 3256 3565 40  0000 L CNN
 F 2 "" H 3288 3500 30  0000 C CNN
 F 3 "" H 3250 3650 60  0000 C CNN
@@
 P 4300 4300
 F 0 "C4" H 4300 4400 40  0000 L CNN
-F 1 "0.1uF" H 4306 4215 40  0000 L CNN
+F 1 "100nF" H 4306 4215 40  0000 L CNN
 F 2 "" H 4338 4150 30  0000 C CNN
 F 3 "" H 4300 4300 60  0000 C CNN
